File: pcb/Bobot_2_Amethyst/Bobot_2_Amethyst.kicad_sch (KiCad schematic)
At the start: 0 parts

Commit message: pcb: add basic elements to esp32 and buttons pcbs
Parts:
- added BatteryIn1: Conn_01x02_Socket, Connector_JST:JST_XH_B2B-XH-A_1x02_P2.50mm_Vertical, symbol Connector:Conn_01x02_Socket
- added BtnBL1: BL, SW_DPDT_XLX:SW_DPDT_XLX, symbol Switch:SW_Push_DPDT
- added BtnBM1: BM, SW_DPDT_XLX:SW_DPDT_XLX, symbol Switch:SW_Push_DPDT
- added BtnBR1: BR, SW_DPDT_XLX:SW_DPDT_XLX, symbol Switch:SW_Push_DPDT
- added BtnBusIn1: BtnBusIn, Connector_JST:JST_XH_B10B-XH-A_1x10_P2.50mm_Vertical, symbol Connector:Conn_01x10_Socket
- added BtnBusOut1: BtnBusOut, Connector_JST:JST_XH_B10B-XH-A_1x10_P2.50mm_Vertical, symbol Connector:Conn_01x10_Socket
- added BtnML1: ML, SW_DPDT_XLX:SW_DPDT_XLX, symbol Switch:SW_Push_DPDT
- added BtnMM1: MM, SW_DPDT_XLX:SW_DPDT_XLX, symbol Switch:SW_Push_DPDT
- added BtnMR1: MR, SW_DPDT_XLX:SW_DPDT_XLX, symbol Switch:SW_Push_DPDT
- added BtnTL1: TL, SW_DPDT_XLX:SW_DPDT_XLX, symbol Switch:SW_Push_DPDT
- added BtnTM1: TM, SW_DPDT_XLX:SW_DPDT_XLX, symbol Switch:SW_Push_DPDT
- added BtnTR1: TR, SW_DPDT_XLX:SW_DPDT_XLX, symbol Switch:SW_Push_DPDT
- added Display_connector1: Conn_01x04_Socket, Connector_JST:JST_XH_B4B-XH-A_1x04_P2.50mm_Vertical, symbol Connector:Conn_01x04_Socket
- added U1: ESP32_DevKit_V1_DOIT, ESP32_DevKit_V1_DOIT:esp32_devkit_v1_doit, symbol ESP32_DevKit_V1_DOIT:ESP32_DevKit_V1_DOIT
Connections:
- new net: BtnBR1.2 (B), BtnBusOut1.10 (BR)
- new net: BtnBusOut1.2 (TL), BtnTL1.2 (B)
- new net: BtnBusOut1.3 (TM), BtnTM1.2 (B)
- new net: BtnBusOut1.4 (TR), BtnTR1.2 (B)
- new net: BtnBusOut1.5 (ML), BtnML1.2 (B)
- new net: BtnBusOut1.6 (MM), BtnMM1.2 (B)
- new net: BtnBusOut1.7 (MR), BtnMR1.2 (B)
- new net: BtnBL1.2 (B), BtnBusOut1.8 (BL)
- new net: BtnBM1.2 (B), BtnBusOut1.9 (BM)
- new net: BtnBusIn1.2 (TL), U1.18 (IO15)
- new net: BtnBusIn1.3 (TM), U1.20 (IO4)
- new net: BtnBusIn1.4 (TR), U1.21 (IO16)
- new net: BtnBusIn1.5 (ML), U1.22 (IO17)
- new net: BtnBusIn1.6 (MM), U1.23 (IO5)
- new net: BtnBusIn1.7 (MR), U1.24 (IO18)
- new net: BtnBusIn1.8 (BL), U1.25 (IO19)
- new net: BtnBusIn1.9 (BM), U1.26 (IO21)
- new net: BtnBusIn1.10 (BR), U1.29 (IO22)
- new net GND: BatteryIn1.1 (GND), BtnBusIn1.1 (GND), Display_connector1.1 (GND), U1.14 (GND), U1.17 (GND)
- new net GND1: BtnBL1.3 (C), BtnBM1.3 (C), BtnBR1.3 (C), BtnBusOut1.1 (GND), BtnML1.3 (C), BtnMM1.3 (C), BtnMR1.3 (C), BtnTL1.3 (C), BtnTM1.3 (C), BtnTR1.3 (C)
- no-connect marks 0 -> 36
Other:
- note added: "Buttons PCB"
